Commit message: srs_model: derive the wrist and carry the distal payload, validated against KDL
Configure the node with only base_link; the wrist is found by walking 7 revolute
joints out from it, enforcing the SRS invariant rather than trusting a hand-entered
tip_link that could disagree. Everything past the wrist (gripper body, fingers,
tools) is lumped at load into the last segment's inertial, so gravity and Coriolis
carry the distal mass: movable distal joints are frozen at the URDF home, and a
rigid attachment is the same rigid body as a bigger last link.

The test fixture is the real OpenArm V1.0 description with the gripper fingers, so
the distal path is exercised by loading it. Validation is against KDL: the serial
ChainDynParam cannot represent the branched gripper, so tools/kdl_reference.cpp
uses KDL's TreeIdSolver_RNE (tree inverse dynamics, fingers pinned at home) to
generate the *_matches_kdl arrays; the implementation matches to <1e-3 on both
arms. Gravity is additionally checked against the potential-energy gradient, and
the distal lump against hand-computed finger values.

File: srs_model/tests/fixtures/openarm_v10.urdf (robot description, URDF)
Before this commit: robot openarm, 20 links, 19 joints
Links:
- added link openarm_left_left_finger, mass 0.03602545343277134; collision mesh filename=package://openarm_description/assets/end_effector/parallel_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 scale=0.001 0.001 0.001; visual mesh filename=package://openarm_description/assets/end_effector/parallel_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 scale=0.001 0.001 0.001
- added link openarm_left_right_finger, mass 0.03602545343277134; collision mesh filename=package://openarm_description/assets/end_effector/parallel_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 scale=0.001 -0.001 0.001; visual mesh filename=package://openarm_description/assets/end_effector/parallel_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 scale=0.001 -0.001 0.001
- added link openarm_right_left_finger, mass 0.03602545343277134; collision mesh filename=package://openarm_description/assets/end_effector/parallel_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 scale=0.001 0.001 0.001; visual mesh filename=package://openarm_description/assets/end_effector/parallel_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 scale=0.001 0.001 0.001
- added link openarm_right_right_finger, mass 0.03602545343277134; collision mesh filename=package://openarm_description/assets/end_effector/parallel_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 scale=0.001 -0.001 0.001; visual mesh filename=package://openarm_description/assets/end_effector/parallel_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 scale=0.001 -0.001 0.001
Joints:
- added joint openarm_left_finger_joint1: type prismatic, parent openarm_left_link7, child openarm_left_right_finger, origin xyz=0.0 0.0 0.1025 rpy=0 0 0, axis 0 -1 0, limit lower=0.0 upper=0.044 effort=333 velocity=10.0
- added joint openarm_left_finger_joint2: type prismatic, parent openarm_left_link7, child openarm_left_left_finger, origin xyz=0.0 -0.0 0.1025 rpy=0 0 0, axis 0 1 0, limit lower=0.0 upper=0.044 effort=333 velocity=10.0, mimic joint=openarm_left_finger_joint1
- added joint openarm_right_finger_joint1: type prismatic, parent openarm_right_link7, child openarm_right_right_finger, origin xyz=0.0 0.0 0.1025 rpy=0 0 0, axis 0 -1 0, limit lower=0.0 upper=0.044 effort=333 velocity=10.0
- added joint openarm_right_finger_joint2: type prismatic, parent openarm_right_link7, child openarm_right_left_finger, origin xyz=0.0 -0.0 0.1025 rpy=0 0 0, axis 0 1 0, limit lower=0.0 upper=0.044 effort=333 velocity=10.0, mimic joint=openarm_right_finger_joint1
